File: lightblade-rev1.kicad_pcb (KiCad board)
At the start: 2 copper layers, 99.1 x 43.2 mm, 17 parts, among them P1 CONN_01X03, P2 CONN_01X02, P3 CONN_02X08, P4 CONN_01X06, U3 Teensy_3.1, U4 74HCT245

Commit message: Final commit before project archive
Routing:
- net VCC: track 0.00 -> 102.1 mm
- net /AUX5: track 0.00 -> 52.2 mm
- net /AUX4: track 0.00 -> 50.3 mm
- net /OCTO7: track 0.00 -> 49.2 mm
- net /AUX2: track 0.00 -> 49.2 mm
- net /AUX3: track 0.00 -> 48.7 mm
- net /OCTO6: track 0.00 -> 45.6 mm
- net /AUX1: track 0.00 -> 45.3 mm
- net /RS-485DE: track 0.00 -> 44.9 mm, vias 0 -> 1
- net /OCTO1: track 0.00 -> 42.6 mm
- net /OCTO8: track 0.00 -> 30.8 mm
- net /OCTO5: track 0.00 -> 29.3 mm
- net /OCTO3: track 0.00 -> 27.8 mm
- net /OCTO4: track 0.00 -> 24.2 mm
- net /RS-485TX: track 0.00 -> 21.8 mm
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- added copper zone on B.Cu, net GND
