File: lightblade-rev1.sch (KiCad schematic (older format))
At the start: 16 parts, among them P1 CONN_01X03, P2 CONN_01X02, P3 CONN_02X08, P4 CONN_01X06, U1 LT1129CST-5, U3 Teensy_3.1, U4 74HCT245

Commit message: updates :/
Parts:
- removed U1: LT1129CST-5, SOT-223, symbol LT1129CST-5
- added C1: 1uF, Capacitors_ThroughHole:C_Disc_D6_P5, symbol CP
- added C2: 0.1uF, Capacitors_ThroughHole:C_Disc_D6_P5, symbol CP
- P1: footprint (none) -> Pin_Headers:Pin_Header_Straight_1x03
- P2: footprint (none) -> Pin_Headers:Pin_Header_Straight_1x02
- P3: footprint (none) -> Pin_Headers:Pin_Header_Straight_2x08
- P4: footprint (none) -> Pin_Headers:Pin_Header_Straight_1x06
- R1, R2, R3, R4, R5, R6, R7, R8: footprint (none) -> Resistors_ThroughHole:Resistor_Horizontal_RM10mm
- RS1: footprint (none) -> Housings_DIP:DIP-8_W7.62mm
- U3: footprint (none) -> Teensy-3:Teensy-3.1
- U4: footprint (none) -> Housings_DIP:DIP-20_W7.62mm
Connections:
- net +12V is gone; now on net VCC: P2.2 (P2)
- net GND: now also C1.2, C2.2
- net OCTO6: now also U3.20 (20/A6); no longer U3.21 (21/A7)
- net OCTO7: now also U3.21 (21/A7); no longer U3.20 (20/A6)
- net VCC: now also C1.1, C2.1
